File: Eagle Files/ArduSensor Shield-v13.brd (EAGLE design)
At the start: 61 x 53.3 mm, 23 parts

Commit message: fixed text and added OSHWA logo
Parts:
- added U$10: (no value), Qtechknow:QTK_GUYMEDIUM
- added U$6: (no value), SparkFun-Aesthetics:SFE_LOGO_FLAME_.3
- added U$7: (no value), Qtechknow:QTK_GUYBIG
- added U$8: (no value), SparkFun-Aesthetics:OSHW-LOGO-M
Routing:
- added copper zone on layer 1, net GND
- added copper zone on layer 16, net GND
Changed lines of the file:
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@@
 <layer number="106" name="bPlate" color="7" fill="1" visible="no" active="no"/>
 <layer number="107" name="Crop" color="7" fill="1" visible="no" active="no"/>
+<layer number="108" name="fp8" color="7" fill="1" visible="no" active="yes"/>
+<layer number="109" name="fp9" color="7" fill="1" visible="no" active="yes"/>
+<layer number="110" name="fp0" color="7" fill="1" visible="no" active="yes"/>
+<layer number="111" name="LPC17xx" color="7" fill="1" visible="yes" active="yes"/>
+<layer number="112" name="tSilk" color="7" fill="1" visible="yes" active="yes"/>
 <layer number="116" name="Patch_BOT" color="9" fill="4" visible="no" active="no"/>
 <layer number="121" name="_tsilk" color="7" fill="1" visible="no" active="no"/>
 <layer number="122" name="_bsilk" color="7" fill="1" visible="no" active="no"/>
+<layer number="123" name="tTestmark" color="7" fill="1" visible="no" active="yes"/>
+<layer number="124" name="bTestmark" color="7" fill="1" visible="no" active="yes"/>
 <layer number="125" name="_tNames" color="7" fill="1" visible="no" active="no"/>
+<layer number="126" name="_bNames" color="7" fill="1" visible="yes" active="yes"/>
+<layer number="127" name="_tValues" color="7" fill="1" visible="yes" active="yes"/>
+<layer number="128" name="_bValues" color="7" fill="1" visible="yes" active="yes"/>
+<layer number="131" name="tAdjust" color="7" fill="1" visible="no" active="yes"/>
+<layer number="132" name="bAdjust" color="7" fill="1" visible="no" active="yes"/>
 <layer number="144" name="Drill_legend" color="7" fill="1" visible="no" active="no"/>
 <layer number="151" name="HeatSink" color="7" fill="1" visible="no" active="no"/>
+<layer number="152" name="_bDocu" color="7" fill="1" visible="yes" active="yes"/>
+<layer number="199" name="Contour" color="7" fill="1" visible="yes" active="yes"/>
 <layer number="200" name="200bmp" color="1" fill="10" visible="no" active="no"/>
 <layer number="201" name="201bmp" color="2" fill="10" visible="no" active="no"/>
@@
 <layer number="223" name="223bmp" color="24" fill="1" visible="no" active="no"/>
 <layer number="224" name="224bmp" color="25" fill="1" visible="no" active="no"/>
+<layer number="248" name="Housing" color="7" fill="1" visible="yes" active="yes"/>
+<layer number="249" name="Edge" color="7" fill="1" visible="yes" active="yes"/>
 <layer number="250" name="Descript" color="3" fill="1" visible="no" active="no"/>
 <layer number="251" name="SMDround" color="12" fill="11" visible="no" active="no"/>
@@
 <text x="22.86" y="33.655" size="0.8128" layer="21" font="vector" ratio="16" align="center">330</text>
 <text x="15.24" y="33.655" size="0.8128" layer="21" font="vector" ratio="16" align="center">330</text>
+<text x="43.18" y="16.51" size="2.1844" layer="21" ratio="16" align="center">+</text>
 </plain>
 <attributes>
@@
 <element name="JP9" library="SparkFun-Aesthetics" package="SFE-NEW-WEBLOGO" value="LOGO-SFENEW" x="16.51" y="5.969" rot="R90"/>
 <element name="FRAME1" library="SparkFun-Aesthetics" package="CREATIVE_COMMONS" value="FRAME-LETTER" x="19.05" y="-19.05"/>
+<element name="U$7" library="Qtechknow" package="QTK_GUYBIG" value="" x="34.29" y="15.24" rot="MR0"/>
+<element name="U$8" library="SparkFun-Aesthetics" package="OSHW-LOGO-M" value="" x="20.32" y="15.24" rot="R90"/>
+<element name="U$10" library="Qtechknow" package="QTK_GUYMEDIUM" value="" x="41.91" y="12.7" rot="R90"/>
+<element name="U$6" library="SparkFun-Aesthetics" package="SFE_LOGO_FLAME_.3" value="" x="45.72" y="17.78" rot="R90"/>
 </elements>
 <signals>
@@
 <wire x1="27.94" y1="20.32" x2="12.7" y2="20.32" width="0.4064" layer="16"/>
 <wire x1="12.7" y1="20.32" x2="3.81" y2="29.21" width="0.4064" layer="16"/>
+<polygon width="0.4064" layer="1" isolate="0.3048">
+<vertex x="0" y="53.34"/>
+<vertex x="58.42" y="53.34"/>
+<vertex x="58.42" y="40.64"/>
+<vertex x="60.96" y="38.1"/>
+<vertex x="60.96" y="5.08"/>
+<vertex x="58.42" y="2.54"/>
+<vertex x="58.42" y="0"/>
+<vertex x="0" y="0"/>
+</polygon>
+<polygon width="0.4064" layer="16" isolate="0.3048">
+<vertex x="0" y="53.34"/>
+<vertex x="58.42" y="53.34"/>
+<vertex x="58.42" y="40.64"/>
+<vertex x="60.96" y="38.1"/>
+<vertex x="60.96" y="5.08"/>
+<vertex x="58.42" y="2.54"/>
+<vertex x="58.42" y="0"/>
+<vertex x="0" y="0"/>
+</polygon>
 </signal>
 <signal name="5V">
