File: Eagle Files/SensorBoard-v13.sch (EAGLE design)
At the start: 40 parts, among them U2 METHANE_SENSOR

Commit message: added better Qtechknow logo dude to the boards
Parts:
- removed U2: METHANE_SENSOR, 1_SparkFun-Sensors:METHANE_SENSOR
- added U$1: GAS-SENSORNEW, Qtechknow:GAS-SENSORNEW
- renumbered 1_R1 to R8
Connections:
- net 1_N$1: now also U$1.A1; no longer U2.A1
- net 1_N$2: now also U$1.B1, U$1.B2, U$1.HB; no longer U2.B1, U2.B2, U2.HB
- net 1_N$3: now also U$1.HA; no longer U2.HA
- net 1_N$4: now also U$1.A2; no longer U2.A2
Changed lines of the file:
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@@
 <?xml version="1.0" encoding="utf-8"?>
 <!DOCTYPE eagle SYSTEM "eagle.dtd">
-<eagle version="6.5.0">
+<eagle version="7.0.0">
 <drawing>
 <settings>
@@
 <layer number="54" name="bGND_GNDA" color="1" fill="9" visible="no" active="no"/>
 <layer number="56" name="wert" color="7" fill="1" visible="no" active="no"/>
+<layer number="57" name="tCAD" color="7" fill="1" visible="no" active="no"/>
+<layer number="59" name="tCarbon" color="7" fill="1" visible="no" active="no"/>
+<layer number="60" name="bCarbon" color="7" fill="1" visible="no" active="no"/>
 <layer number="91" name="Nets" color="2" fill="1" visible="yes" active="yes"/>
 <layer number="92" name="Busses" color="1" fill="1" visible="yes" active="yes"/>
@@
 <layer number="97" name="Info" color="7" fill="1" visible="yes" active="yes"/>
 <layer number="98" name="Guide" color="6" fill="1" visible="yes" active="yes"/>
+<layer number="99" name="SpiceOrder" color="7" fill="1" visible="no" active="no"/>
 <layer number="100" name="Muster" color="7" fill="1" visible="no" active="no"/>
 <layer number="101" name="Patch_Top" color="12" fill="4" visible="no" active="yes"/>
@@
 <layer number="106" name="bPlate" color="7" fill="1" visible="no" active="yes"/>
 <layer number="107" name="Crop" color="7" fill="1" visible="no" active="yes"/>
+<layer number="108" name="fp8" color="7" fill="1" visible="no" active="yes"/>
+<layer number="109" name="fp9" color="7" fill="1" visible="no" active="yes"/>
+<layer number="110" name="fp0" color="7" fill="1" visible="no" active="yes"/>
+<layer number="111" name="LPC17xx" color="7" fill="1" visible="yes" active="yes"/>
+<layer number="112" name="tSilk" color="7" fill="1" visible="yes" active="yes"/>
+<layer number="113" name="IDFDebug" color="4" fill="1" visible="yes" active="yes"/>
 <layer number="116" name="Patch_BOT" color="9" fill="4" visible="no" active="yes"/>
 <layer number="121" name="_tsilk" color="7" fill="1" visible="no" active="yes"/>
 <layer number="122" name="_bsilk" color="7" fill="1" visible="no" active="yes"/>
+<layer number="123" name="tTestmark" color="7" fill="1" visible="no" active="yes"/>
+<layer number="124" name="bTestmark" color="7" fill="1" visible="no" active="yes"/>
 <layer number="125" name="_tNames" color="7" fill="1" visible="no" active="yes"/>
+<layer number="126" name="_bNames" color="7" fill="1" visible="yes" active="yes"/>
+<layer number="127" name="_tValues" color="7" fill="1" visible="yes" active="yes"/>
+<layer number="128" name="_bValues" color="7" fill="1" visible="yes" active="yes"/>
+<layer number="129" name="Mask" color="7" fill="1" visible="no" active="yes"/>
+<layer number="131" name="tAdjust" color="7" fill="1" visible="no" active="yes"/>
+<layer number="132" name="bAdjust" color="7" fill="1" visible="no" active="yes"/>
 <layer number="144" name="Drill_legend" color="7" fill="1" visible="no" active="yes"/>
+<layer number="150" name="Notes" color="7" fill="1" visible="yes" active="yes"/>
 <layer number="151" name="HeatSink" color="7" fill="1" visible="no" active="yes"/>
+<layer number="152" name="_bDocu" color="7" fill="1" visible="yes" active="yes"/>
+<layer number="153" name="FabDoc1" color="7" fill="1" visible="yes" active="yes"/>
+<layer number="154" name="FabDoc2" color="7" fill="1" visible="yes" active="yes"/>
+<layer number="155" name="FabDoc3" color="7" fill="1" visible="yes" active="yes"/>
+<layer number="199" name="Contour" color="7" fill="1" visible="yes" active="yes"/>
 <layer number="200" name="200bmp" color="1" fill="10" visible="no" active="yes"/>
 <layer number="201" name="201bmp" color="2" fill="10" visible="no" active="yes"/>
@@
 <layer number="223" name="223bmp" color="24" fill="1" visible="no" active="no"/>
 <layer number="224" name="224bmp" color="25" fill="1" visible="no" active="no"/>
+<layer number="248" name="Housing" color="7" fill="1" visible="yes" active="yes"/>
+<layer number="249" name="Edge" color="7" fill="1" visible="yes" active="yes"/>
 <layer number="250" name="Descript" color="3" fill="1" visible="no" active="no"/>
 <layer number="251" name="SMDround" color="12" fill="11" visible="no" active="no"/>
@@
 </classes>
 <parts>
-<part name="U2" library="1_SparkFun-Sensors" deviceset="METHANE_SENSOR" device=""/>
-<part name="1_R1" library="1_SparkFun-Passives" deviceset="RESISTOR" device="AXIAL-0.3"/>
+<part name="R8" library="1_SparkFun-Passives" deviceset="RESISTOR" device="AXIAL-0.3"/>
 <part name="JP8" library="1_SparkFun-Connectors" deviceset="M01" device="PTH" value=""/>
 <part name="JP16" library="1_SparkFun-Connectors" deviceset="M04" device="PTH"/>
@@
 <part name="LOGO7" library="SparkFun-Aesthetics" deviceset="LOGO-SFE" device="SK"/>
 <part name="LOGO8" library="SparkFun-Aesthetics" deviceset="LOGO-SFE" device="SK"/>
+<part name="U$1" library="Qtechknow" deviceset="GAS-SENSORNEW" device=""/>
 </parts>
 <sheets>
@@
 </plain>
 <instances>
-<instance part="U2" gate="G$1" x="-58.42" y="127"/>
-<instance part="1_R1" gate="G$1" x="-73.66" y="114.3" rot="R270"/>
+<instance part="R8" gate="G$1" x="-73.66" y="114.3" rot="R270"/>
 <instance part="JP8" gate="G$1" x="-96.52" y="132.08"/>
 <instance part="JP16" gate="G$1" x="-93.98" y="109.22" rot="MR180"/>
@@
 <instance part="LOGO7" gate="G$1" x="-5.08" y="30.48"/>
 <instance part="LOGO8" gate="G$1" x="-5.08" y="22.86"/>
+<instance part="U$1" gate="G$1" x="-58.42" y="127"/>
 </instances>
 <busses>
@@
 <segment>
 <pinref part="JP8" gate="G$1" pin="1"/>
-<pinref part="U2" gate="G$1" pin="A1"/>
 <wire x1="-88.9" y1="132.08" x2="-71.12" y2="132.08" width="0.1524" layer="91"/>
+<pinref part="U$1" gate="G$1" pin="A1"/>
 </segment>
 </net>
@@
 <wire x1="-88.9" y1="104.14" x2="-40.64" y2="104.14" width="0.1524" layer="91"/>
 <wire x1="-40.64" y1="104.14" x2="-40.64" y2="121.92" width="0.1524" layer="91"/>
-<pinref part="U2" gate="G$1" pin="B1"/>
 <wire x1="-40.64" y1="121.92" x2="-40.64" y2="127" width="0.1524" layer="91"/>
 <wire x1="-40.64" y1="127" x2="-40.64" y2="132.08" width="0.1524" layer="91"/>
 <wire x1="-40.64" y1="132.08" x2="-45.72" y2="132.08" width="0.1524" layer="91"/>
-<pinref part="U2" gate="G$1" pin="HB"/>
 <wire x1="-43.18" y1="127" x2="-40.64" y2="127" width="0.1524" layer="91"/>
 <junction x="-40.64" y="127"/>
-<pinref part="U2" gate="G$1" pin="B2"/>
 <wire x1="-45.72" y1="121.92" x2="-40.64" y2="121.92" width="0.1524" layer="91"/>
 <junction x="-40.64" y="121.92"/>
+<pinref part="U$1" gate="G$1" pin="HB"/>
+<pinref part="U$1" gate="G$1" pin="B1"/>
+<pinref part="U$1" gate="G$1" pin="B2"/>
 </segment>
 </net>
@@
 <wire x1="-81.28" y1="106.68" x2="-81.28" y2="109.22" width="0.1524" layer="91"/>
 <junction x="-81.28" y="106.68"/>
-<pinref part="U2" gate="G$1" pin="HA"/>
 <wire x1="-81.28" y1="109.22" x2="-81.28" y2="127" width="0.1524" layer="91"/>
 <wire x1="-81.28" y1="127" x2="-73.66" y2="127" width="0.1524" layer="91"/>
@@
 <wire x1="-88.9" y1="109.22" x2="-81.28" y2="109.22" width="0.1524" layer="91"/>
 <junction x="-81.28" y="109.22"/>
-<pinref part="1_R1" gate="G$1" pin="2"/>
+<pinref part="R8" gate="G$1" pin="2"/>
 <wire x1="-73.66" y1="109.22" x2="-73.66" y2="106.68" width="0.1524" layer="91"/>
+<pinref part="U$1" gate="G$1" pin="HA"/>
 </segment>
 </net>
 <net name="1_N$4" class="0">
 <segment>
-<pinref part="U2" gate="G$1" pin="A2"/>
 <wire x1="-71.12" y1="121.92" x2="-73.66" y2="121.92" width="0.1524" layer="91"/>
-<pinref part="1_R1" gate="G$1" pin="1"/>
+<pinref part="R8" gate="G$1" pin="1"/>
 <wire x1="-73.66" y1="121.92" x2="-73.66" y2="119.38" width="0.1524" layer="91"/>
+<pinref part="U$1" gate="G$1" pin="A2"/>
 </segment>
 </net>
@@
 </sheet>
 </sheets>
+<errors>
+</errors>
 </schematic>
 </drawing>
